File: hardware/Sandwich.sch (KiCad schematic (older format))
At the start: 19 parts

Commit message: Updated schematics.
Parts:
- removed Q?: PN2222A, symbol Q_NPN_BCE
- added P1: CONN_01X20, Pin_Headers:Pin_Header_Straight_1x20, symbol CONN_01X20
- added P2: CONN_01X06, Pin_Headers:Pin_Header_Straight_1x06, symbol CONN_01X06
- added Q1: PZT2222A, TO_SOT_Packages_SMD:SOT-223, symbol PZT2222A
- ??1: renamed from ???; footprint (none) -> Housings_DIP:DIP-40_W15.24mm_LongPads
- C1: renamed from C?; footprint (none) -> Capacitors_ThroughHole:C_Disc_D3_P2.5
- D1: renamed from D?; footprint (none) -> LEDs:LED-3MM
- P3: renamed from P?; footprint (none) -> libraries:conn_SPC15430
- R1, R10, R11, R2, R3, R4, R5, R6, R7, R8, R9: renamed from R?; footprint (none) -> Resistors_ThroughHole:Resistor_Horizontal_RM10mm
- U1: renamed from U?; footprint (none) -> Housings_DIP:DIP-8_W7.62mm_LongPads
- Y1: renamed from Y?; footprint (none) -> Crystals:Crystal_HC49-U_Vertical
Connections:
- net PROP_TX is gone; now on net PROP_RX: ??1.39 (P30)
- net 3.3V: now also P2.2 (P2)
- net 5V: now also P2.1 (P1)
- net GND: now also P2.6 (P6), Q1.3 (E)
- net PROP_DTR: now also P2.5 (P5)
- net PROP_RX: now also ??1.34 (P25), P1.19 (P19), P2.3 (P3), P2.4 (P4)
- net at ??1.1 (P0): now also P1.16 (P16)
- net at ??1.11 (RES/): now also Q1.2 (C)
- net at ??1.13 (P8): now also P1.8 (P8)
- net at ??1.14 (P9): now also P1.7 (P7)
- net at ??1.15 (P10): now also P1.6 (P6)
- net at ??1.16 (P11): now also P1.5 (P5)
- net at ??1.17 (P12): now also P1.4 (P4)
- net at ??1.18 (P13): now also P1.3 (P3)
- net at ??1.19 (P14): now also P1.2 (P2)
- net at ??1.2 (P1): now also P1.15 (P15)
- net at ??1.20 (P15): now also P1.1 (P1)
- net at ??1.3 (P2): now also P1.14 (P14)
- net at ??1.33 (P24): now also P1.20 (P20)
- net at ??1.35 (P26): now also P1.18 (P18)
- net at ??1.36 (P27): now also P1.17 (P17)
- net at ??1.4 (P3): now also P1.13 (P13)
- net at ??1.5 (P4): now also P1.12 (P12)
- net at ??1.6 (P5): now also P1.11 (P11)
- net at ??1.7 (P6): now also P1.10 (P10)
- net at ??1.8 (P7): now also P1.9 (P9)
- net at C1.1, R1.2: now also Q1.1 (B)
Changed lines of the file:
@@
 $EndDescr
 $Comp
-L P8X32A-D40 ???
+L P8X32A-D40 ??1
 U 2 1 56B3D7DA
 P 9050 4650
-F 0 "???" H 9100 5703 60  0000 C CNN
+F 0 "??1" H 9100 5703 60  0000 C CNN
 F 1 "P8X32A-D40" H 9100 5603 60  0000 C CNN
-F 2 "" H 9050 4650 60  0000 C CNN
+F 2 "Housings_DIP:DIP-40_W15.24mm_LongPads" H 9050 4650 60  0001 C CNN
 F 3 "" H 9050 4650 60  0000 C CNN
 	2    9050 4650
@@
 $EndComp
 $Comp
-L CONN_01X15 P?
+L CONN_01X15 P3
 U 1 1 56B3D8DB
 P 11100 4750
-F 0 "P?" H 10850 3850 50  0000 L CNN
+F 0 "P3" H 10850 3850 50  0000 L CNN
 F 1 "VGA_OUT" H 10850 3950 50  0000 L CNN
-F 2 "" H 11100 4750 50  0000 C CNN
+F 2 "libraries:conn_SPC15430" H 11100 4750 50  0001 C CNN
 F 3 "" H 11100 4750 50  0000 C CNN
 	1    11100 4750
@@
 $EndComp
 $Comp
-L R R?
+L R R7
 U 1 1 56B3DA31
 P 10000 5350
-F 0 "R?" V 10050 5200 50  0000 C CNN
+F 0 "R7" V 10050 5200 50  0000 C CNN
 F 1 "240" V 10000 5350 50  0000 C CNN
-F 2 "" V 9930 5350 50  0000 C CNN
+F 2 "Resistors_ThroughHole:Resistor_Horizontal_RM10mm" V 9930 5350 50  0001 C CNN
 F 3 "" H 10000 5350 50  0000 C CNN
 	1    10000 5350
@@
 $EndComp
 $Comp
-L R R?
+L R R11
 U 1 1 56B3DA8C
 P 10250 5250
-F 0 "R?" V 10300 5400 50  0000 C CNN
+F 0 "R11" V 10300 5400 50  0000 C CNN
 F 1 "240" V 10250 5250 50  0000 C CNN
-F 2 "" V 10180 5250 50  0000 C CNN
+F 2 "Resistors_ThroughHole:Resistor_Horizontal_RM10mm" V 10180 5250 50  0001 C CNN
 F 3 "" H 10250 5250 50  0000 C CNN
 	1    10250 5250
@@
 	9750 5250 10100 5250
 $Comp
-L R R?
+L R R6
 U 1 1 56B3DB9A
 P 10000 5150
-F 0 "R?" V 10050 5000 50  0000 C CNN
+F 0 "R6" V 10050 5000 50  0000 C CNN
 F 1 "470" V 10000 5150 50  0000 C CNN
-F 2 "" V 9930 5150 50  0000 C CNN
+F 2 "Resistors_ThroughHole:Resistor_Horizontal_RM10mm" V 9930 5150 50  0001 C CNN
 F 3 "" H 10000 5150 50  0000 C CNN
 	1    10000 5150
@@
 $EndComp
 $Comp
-L R R?
+L R R10
 U 1 1 56B3DBE5
 P 10250 5050
-F 0 "R?" V 10300 5200 50  0000 C CNN
+F 0 "R10" V 10300 5200 50  0000 C CNN
 F 1 "240" V 10250 5050 50  0000 C CNN
-F 2 "" V 10180 5050 50  0000 C CNN
+F 2 "Resistors_ThroughHole:Resistor_Horizontal_RM10mm" V 10180 5050 50  0001 C CNN
 F 3 "" H 10250 5050 50  0000 C CNN
 	1    10250 5050
@@
 	9750 5050 10100 5050
 $Comp
-L R R?
+L R R5
 U 1 1 56B3DEC9
 P 10000 4950
-F 0 "R?" V 10050 4800 50  0000 C CNN
+F 0 "R5" V 10050 4800 50  0000 C CNN
 F 1 "470" V 10000 4950 50  0000 C CNN
-F 2 "" V 9930 4950 50  0000 C CNN
+F 2 "Resistors_ThroughHole:Resistor_Horizontal_RM10mm" V 9930 4950 50  0001 C CNN
 F 3 "" H 10000 4950 50  0000 C CNN
 	1    10000 4950
@@
 $EndComp
 $Comp
-L R R?
+L R R9
 U 1 1 56B3DF20
 P 10250 4850
-F 0 "R?" V 10300 5000 50  0000 C CNN
+F 0 "R9" V 10300 5000 50  0000 C CNN
 F 1 "240" V 10250 4850 50  0000 C CNN
-F 2 "" V 10180 4850 50  0000 C CNN
+F 2 "Resistors_ThroughHole:Resistor_Horizontal_RM10mm" V 10180 4850 50  0001 C CNN
 F 3 "" H 10250 4850 50  0000 C CNN
 	1    10250 4850
@@
 	10100 4850 9750 4850
 $Comp
-L R R?
+L R R4
 U 1 1 56B3E13C
 P 10000 4750
-F 0 "R?" V 10050 4600 50  0000 C CNN
+F 0 "R4" V 10050 4600 50  0000 C CNN
 F 1 "470" V 10000 4750 50  0000 C CNN
-F 2 "" V 9930 4750 50  0000 C CNN
+F 2 "Resistors_ThroughHole:Resistor_Horizontal_RM10mm" V 9930 4750 50  0001 C CNN
 F 3 "" H 10000 4750 50  0000 C CNN
 	1    10000 4750
@@
 $EndComp
 $Comp
-L R R?
+L R R8
 U 1 1 56B3E18E
 P 10250 4650
-F 0 "R?" V 10300 4800 50  0000 C CNN
+F 0 "R8" V 10300 4800 50  0000 C CNN
 F 1 "240" V 10250 4650 50  0000 C CNN
-F 2 "" V 10180 4650 50  0000 C CNN
+F 2 "Resistors_ThroughHole:Resistor_Horizontal_RM10mm" V 10180 4650 50  0001 C CNN
 F 3 "" H 10250 4650 50  0000 C CNN
 	1    10250 4650
@@
 Connection ~ 10500 4650
 $Comp
-L Crystal_Small Y?
+L Crystal_Small Y1
 U 1 1 56B3E76F
 P 10000 5550
-F 0 "Y?" H 10000 5650 50  0000 C CNN
+F 0 "Y1" H 10000 5650 50  0000 C CNN
 F 1 "5MHz" H 10000 5400 50  0000 C CNN
-F 2 "" H 10000 5550 50  0000 C CNN
+F 2 "Crystals:Crystal_HC49-U_Vertical" H 10000 5550 50  0001 C CNN
 F 3 "" H 10000 5550 50  0000 C CNN
 	1    10000 5550
@@
 	10150 5550 10100 5550
 $Comp
-L 24C512 U?
+L 24C512 U1
 U 1 1 56B3EA78
 P 9050 2600
-F 0 "U?" H 9050 3266 50  0000 C CNN
+F 0 "U1" H 9050 3266 50  0000 C CNN
 F 1 "24C512" H 9050 3166 50  0000 C CNN
-F 2 "" H 9050 2600 50  0000 C CNN
+F 2 "Housings_DIP:DIP-8_W7.62mm_LongPads" H 9050 2600 50  0001 C CNN
 F 3 "" H 9050 2600 50  0000 C CNN
 	1    9050 2600
@@
 $EndComp
 $Comp
-L P8X32A-D40 ???
+L P8X32A-D40 ??1
 U 1 1 56B5DEF4
 P 7900 2600
-F 0 "???" H 7850 3008 60  0000 C CNN
+F 0 "??1" H 7850 3008 60  0000 C CNN
 F 1 "P8X32A-D40" H 7850 2900 60  0000 C CNN
-F 2 "" H 7900 2600 60  0000 C CNN
+F 2 "Housings_DIP:DIP-40_W15.24mm_LongPads" H 7900 2600 60  0001 C CNN
 F 3 "" H 7900 2600 60  0000 C CNN
 	1    7900 2600
@@
 	10750 4850 10900 4850
 $Comp
-L R R?
+L R R3
 U 1 1 56B5E9EC
 P 9550 1950
-F 0 "R?" V 9355 1950 50  0000 C CNN
+F 0 "R3" V 9355 1950 50  0000 C CNN
 F 1 "10k" V 9455 1950 50  0000 C CNN
-F 2 "" V 9480 1950 50  0000 C CNN
+F 2 "Resistors_ThroughHole:Resistor_Horizontal_RM10mm" V 9480 1950 50  0001 C CNN
 F 3 "" H 9550 1950 50  0000 C CNN
 	1    9550 1950
@@
 	7400 1950 7400 2600
 $Comp
-L LED D?
+L LED D1
 U 1 1 56B5F331
 P 7400 2800
-F 0 "D?" V 7450 2692 50  0000 R CNN
+F 0 "D1" V 7450 2692 50  0000 R CNN
 F 1 "LED" V 7350 2692 50  0000 R CNN
-F 2 "" H 7400 2800 50  0000 C CNN
+F 2 "LEDs:LED-3MM" H 7400 2800 50  0001 C CNN
 F 3 "" H 7400 2800 50  0000 C CNN
 	1    7400 2800
@@
 $EndComp
 $Comp
-L R R?
+L R R2
 U 1 1 56B5F44A
 P 7850 3100
-F 0 "R?" V 7655 3100 50  0000 C CNN
+F 0 "R2" V 7655 3100 50  0000 C CNN
 F 1 "1.5k" V 7755 3100 50  0000 C CNN
-F 2 "" V 7780 3100 50  0000 C CNN
+F 2 "Resistors_ThroughHole:Resistor_Horizontal_RM10mm" V 7780 3100 50  0001 C CNN
 F 3 "" H 7850 3100 50  0000 C CNN
 	1    7850 3100
@@
 	8300 5550 8450 5550
 $Comp
-L R R?
+L R R1
 U 1 1 56B7C3FF
 P 7650 6300
-F 0 "R?" V 7455 6300 50  0000 C CNN
+F 0 "R1" V 7455 6300 50  0000 C CNN
 F 1 "10k" V 7555 6300 50  0000 C CNN
-F 2 "" V 7580 6300 50  0000 C CNN
+F 2 "Resistors_ThroughHole:Resistor_Horizontal_RM10mm" V 7580 6300 50  0001 C CNN
 F 3 "" H 7650 6300 50  0000 C CNN
 	1    7650 6300
 	0    1    1    0
-$EndComp
-$Comp
-L Q_NPN_BCE Q?
-U 1 1 56B7C5EC
-P 7950 5950
-F 0 "Q?" H 8144 6000 50  0000 L CNN
-F 1 "PN2222A" H 8144 5900 50  0000 L CNN
-F 2 "" H 8150 6050 50  0000 C CNN
-F 3 "" H 7950 5950 50  0000 C CNN
-	1    7950 5950
-	1    0    0    -1
 $EndComp
 Text GLabel 8350 6300 2    60   Input ~ 0
@@
 	8050 5750 8050 5650
 $Comp
-L C C?
+L C C1
 U 1 1 56B7CB28
 P 7050 5950
-F 0 "C?" V 6810 5950 50  0000 C CNN
+F 0 "C1" V 6810 5950 50  0000 C CNN
 F 1 "10nF" V 6910 5950 50  0000 C CNN
-F 2 "" H 7088 5800 50  0000 C CNN
+F 2 "Capacitors_ThroughHole:C_Disc_D3_P2.5" H 7088 5800 50  0001 C CNN
 F 3 "" H 7050 5950 50  0000 C CNN
 	1    7050 5950
@@
 	6600 5950 6900 5950
 Connection ~ 7400 5950
+Wire Wire Line
+	6950 5350 8450 5350
+Wire Wire Line
+	8450 5250 6950 5250
+Wire Wire Line
+	6950 5150 8450 5150
+Wire Wire Line
+	8450 5050 6950 5050
+Wire Wire Line
+	6950 4950 8450 4950
+Wire Wire Line
+	8450 4850 6950 4850
+Wire Wire Line
+	6950 4750 8450 4750
+Wire Wire Line
+	6950 4650 8450 4650
+Wire Wire Line
+	8450 4550 6950 4550
+Wire Wire Line
+	6950 4450 8450 4450
+Wire Wire Line
+	8450 4350 6950 4350
+Wire Wire Line
+	6950 4250 8450 4250
+Wire Wire Line
+	8450 4150 6950 4150
+Wire Wire Line
+	6950 4050 8450 4050
+Wire Wire Line
+	8450 3950 6950 3950
+Wire Wire Line
+	6950 3850 8450 3850
+Wire Wire Line
+	6950 3750 8600 3750
+Wire Wire Line
+	8600 3750 8600 3700
+Wire Wire Line
+	8600 3700 9800 3700
+Wire Wire Line
+	9800 3700 9800 4250
+Wire Wire Line
+	9800 4250 9750 4250
+Wire Wire Line
+	6950 3650 9950 3650
+Wire Wire Line
+	9950 3650 9950 4350
+Wire Wire Line
+	9950 4350 9750 4350
+Wire Wire Line
+	6950 3550 10000 3550
+Wire Wire Line
+	10000 3550 10000 4450
+Wire Wire Line
+	10000 4450 9750 4450
+Wire Wire Line
+	6950 3450 10050 3450
+Wire Wire Line
+	10050 3450 10050 4550
+Wire Wire Line
+	10050 4550 9750 4550
+$Comp
+L CONN_01X20 P1
+U 1 1 56BE773D
+P 6750 4400
+F 0 "P1" H 6669 3231 50  0000 C CNN
+F 1 "CONN_01X20" H 6669 3331 50  0000 C CNN
+F 2 "Pin_Headers:Pin_Header_Straight_1x20" H 6750 4400 50  0001 C CNN
+F 3 "" H 6750 4400 50  0000 C CNN
+	1    6750 4400
+	-1   0    0    1
+$EndComp
+$Comp
+L CONN_01X06 P2
+U 1 1 56BE77EE
+P 11050 1600
+F 0 "P2" H 11127 1642 50  0000 L CNN
+F 1 "CONN_01X06" H 11127 1542 50  0000 L CNN
+F 2 "Pin_Headers:Pin_Header_Straight_1x06" H 11050 1600 50  0001 C CNN
+F 3 "" H 11050 1600 50  0000 C CNN
+	1    11050 1600
+	1    0    0    -1
+$EndComp
+Text GLabel 10700 1850 0    60   Input ~ 0
+GND
+Text GLabel 10350 1750 0    60   Input ~ 0
+PROP_DTR
+Text GLabel 10700 1650 0    60   Input ~ 0
+PROP_RX
+Text GLabel 10350 1550 0    60   Input ~ 0
+PROP_TX
+Text GLabel 10700 1450 0    60   Input ~ 0
+3.3V
+Text GLabel 10350 1350 0    60   Input ~ 0
+5V
+Wire Wire Line
+	10700 1850 10850 1850
+Wire Wire Line
+	10850 1750 10350 1750
+Wire Wire Line
+	10700 1650 10850 1650
+Wire Wire Line
+	10850 1550 10350 1550
+Wire Wire Line
+	10700 1450 10850 1450
+Wire Wire Line
+	10850 1350 10350 1350
+$Comp
+L PZT2222A Q1
+U 1 1 56BE85CA
+P 7950 5950
+F 0 "Q1" H 8144 6050 50  0000 L CNN
+F 1 "PZT2222A" H 8144 5950 50  0000 L CNN
+F 2 "TO_SOT_Packages_SMD:SOT-223" H 8144 5850 50  0000 L CIN
+F 3 "" H 7950 5950 50  0000 L CNN
+	1    7950 5950
+	1    0    0    -1
+$EndComp
 $EndSCHEMATC

Commit message: Schematics WIP
Parts:
- R1, R10, R11, R2, R3, R4, R5, R6, R7, R8, R9: footprint Resistors_ThroughHole:Resistor_Horizontal_RM10mm -> Resistors_ThroughHole:Resistor_Horizontal_RM15mm
- Y1: footprint Crystals:Crystal_HC49-U_Vertical -> Crystals:Crystal_HC49-U_Horizontal_Typ1
- renumbered ??1 to U1, U1 to U2
Changed lines of the file:
@@
 $EndDescr
 $Comp
-L P8X32A-D40 ??1
+L P8X32A-D40 U1
 U 2 1 56B3D7DA
 P 9050 4650
-F 0 "??1" H 9100 5703 60  0000 C CNN
+F 0 "U1" H 9100 5703 60  0000 C CNN
 F 1 "P8X32A-D40" H 9100 5603 60  0000 C CNN
 F 2 "Housings_DIP:DIP-40_W15.24mm_LongPads" H 9050 4650 60  0001 C CNN
@@
 F 0 "R7" V 10050 5200 50  0000 C CNN
 F 1 "240" V 10000 5350 50  0000 C CNN
-F 2 "Resistors_ThroughHole:Resistor_Horizontal_RM10mm" V 9930 5350 50  0001 C CNN
+F 2 "Resistors_ThroughHole:Resistor_Horizontal_RM15mm" V 9930 5350 50  0001 C CNN
 F 3 "" H 10000 5350 50  0000 C CNN
 	1    10000 5350
@@
 F 0 "R11" V 10300 5400 50  0000 C CNN
 F 1 "240" V 10250 5250 50  0000 C CNN
-F 2 "Resistors_ThroughHole:Resistor_Horizontal_RM10mm" V 10180 5250 50  0001 C CNN
+F 2 "Resistors_ThroughHole:Resistor_Horizontal_RM15mm" V 10180 5250 50  0001 C CNN
 F 3 "" H 10250 5250 50  0000 C CNN
 	1    10250 5250
@@
 F 0 "R6" V 10050 5000 50  0000 C CNN
 F 1 "470" V 10000 5150 50  0000 C CNN
-F 2 "Resistors_ThroughHole:Resistor_Horizontal_RM10mm" V 9930 5150 50  0001 C CNN
+F 2 "Resistors_ThroughHole:Resistor_Horizontal_RM15mm" V 9930 5150 50  0001 C CNN
 F 3 "" H 10000 5150 50  0000 C CNN
 	1    10000 5150
@@
 F 0 "R10" V 10300 5200 50  0000 C CNN
 F 1 "240" V 10250 5050 50  0000 C CNN
-F 2 "Resistors_ThroughHole:Resistor_Horizontal_RM10mm" V 10180 5050 50  0001 C CNN
+F 2 "Resistors_ThroughHole:Resistor_Horizontal_RM15mm" V 10180 5050 50  0001 C CNN
 F 3 "" H 10250 5050 50  0000 C CNN
 	1    10250 5050
@@
 F 0 "R5" V 10050 4800 50  0000 C CNN
 F 1 "470" V 10000 4950 50  0000 C CNN
-F 2 "Resistors_ThroughHole:Resistor_Horizontal_RM10mm" V 9930 4950 50  0001 C CNN
+F 2 "Resistors_ThroughHole:Resistor_Horizontal_RM15mm" V 9930 4950 50  0001 C CNN
 F 3 "" H 10000 4950 50  0000 C CNN
 	1    10000 4950
@@
 F 0 "R9" V 10300 5000 50  0000 C CNN
 F 1 "240" V 10250 4850 50  0000 C CNN
-F 2 "Resistors_ThroughHole:Resistor_Horizontal_RM10mm" V 10180 4850 50  0001 C CNN
+F 2 "Resistors_ThroughHole:Resistor_Horizontal_RM15mm" V 10180 4850 50  0001 C CNN
 F 3 "" H 10250 4850 50  0000 C CNN
 	1    10250 4850
@@
 F 0 "R4" V 10050 4600 50  0000 C CNN
 F 1 "470" V 10000 4750 50  0000 C CNN
-F 2 "Resistors_ThroughHole:Resistor_Horizontal_RM10mm" V 9930 4750 50  0001 C CNN
+F 2 "Resistors_ThroughHole:Resistor_Horizontal_RM15mm" V 9930 4750 50  0001 C CNN
 F 3 "" H 10000 4750 50  0000 C CNN
 	1    10000 4750
@@
 F 0 "R8" V 10300 4800 50  0000 C CNN
 F 1 "240" V 10250 4650 50  0000 C CNN
-F 2 "Resistors_ThroughHole:Resistor_Horizontal_RM10mm" V 10180 4650 50  0001 C CNN
+F 2 "Resistors_ThroughHole:Resistor_Horizontal_RM15mm" V 10180 4650 50  0001 C CNN
 F 3 "" H 10250 4650 50  0000 C CNN
 	1    10250 4650
@@
 	10900 5350 10150 5350
 Wire Wire Line
-	10150 5150 10600 5150
-Wire Wire Line
-	10600 5150 10600 4250
+	10600 5150 10150 5150
+Wire Wire Line
+	10600 4250 10600 5150
 Wire Wire Line
 	10600 4250 10900 4250
@@
 Connection ~ 10600 5050
 Wire Wire Line
-	10150 4950 10550 4950
-Wire Wire Line
-	10550 4950 10550 4150
+	10550 4950 10150 4950
+Wire Wire Line
+	10550 4150 10550 4950
 Wire Wire Line
 	10550 4150 10900 4150
@@
 Connection ~ 10550 4850
 Wire Wire Line
-	10150 4750 10500 4750
-Wire Wire Line
-	10500 4750 10500 4050
+	10500 4750 10150 4750
+Wire Wire Line
+	10500 4050 10500 4750
 Wire Wire Line
 	10500 4050 10900 4050
@@
 F 0 "Y1" H 10000 5650 50  0000 C CNN
 F 1 "5MHz" H 10000 5400 50  0000 C CNN
-F 2 "Crystals:Crystal_HC49-U_Vertical" H 10000 5550 50  0001 C CNN
+F 2 "Crystals:Crystal_HC49-U_Horizontal_Typ1" H 10000 5550 50  0001 C CNN
 F 3 "" H 10000 5550 50  0000 C CNN
 	1    10000 5550
@@
 	10150 5550 10100 5550
 $Comp
-L 24C512 U1
+L 24C512 U2
 U 1 1 56B3EA78
 P 9050 2600
-F 0 "U1" H 9050 3266 50  0000 C CNN
+F 0 "U2" H 9050 3266 50  0000 C CNN
 F 1 "24C512" H 9050 3166 50  0000 C CNN
 F 2 "Housings_DIP:DIP-8_W7.62mm_LongPads" H 9050 2600 50  0001 C CNN
@@
 $EndComp
 $Comp
-L P8X32A-D40 ??1
+L P8X32A-D40 U1
 U 1 1 56B5DEF4
 P 7900 2600
-F 0 "??1" H 7850 3008 60  0000 C CNN
+F 0 "U1" H 7850 3008 60  0000 C CNN
 F 1 "P8X32A-D40" H 7850 2900 60  0000 C CNN
 F 2 "Housings_DIP:DIP-40_W15.24mm_LongPads" H 7900 2600 60  0001 C CNN
@@
 $EndComp
 Wire Wire Line
-	8350 2400 8200 2400
+	8200 2400 8350 2400
 Wire Wire Line
 	8200 2500 8350 2500
@@
 GND
 Wire Wire Line
-	10600 6000 10800 6000
-Wire Wire Line
-	10800 6000 10800 4450
+	10800 6000 10600 6000
+Wire Wire Line
+	10800 4450 10800 6000
 Wire Wire Line
 	10800 4450 10900 4450
@@
 F 0 "R3" V 9355 1950 50  0000 C CNN
 F 1 "10k" V 9455 1950 50  0000 C CNN
-F 2 "Resistors_ThroughHole:Resistor_Horizontal_RM10mm" V 9480 1950 50  0001 C CNN
+F 2 "Resistors_ThroughHole:Resistor_Horizontal_RM15mm" V 9480 1950 50  0001 C CNN
 F 3 "" H 9550 1950 50  0000 C CNN
 	1    9550 1950
@@
 F 0 "R2" V 7655 3100 50  0000 C CNN
 F 1 "1.5k" V 7755 3100 50  0000 C CNN
-F 2 "Resistors_ThroughHole:Resistor_Horizontal_RM10mm" V 7780 3100 50  0001 C CNN
+F 2 "Resistors_ThroughHole:Resistor_Horizontal_RM15mm" V 7780 3100 50  0001 C CNN
 F 3 "" H 7850 3100 50  0000 C CNN
 	1    7850 3100
@@
 	7400 3100 7700 3100
 Connection ~ 8300 3100
-Wire Wire Line
-	9050 2100 9050 1950
 Wire Wire Line
 	9750 3100 9750 2500
@@
 F 0 "R1" V 7455 6300 50  0000 C CNN
 F 1 "10k" V 7555 6300 50  0000 C CNN
-F 2 "Resistors_ThroughHole:Resistor_Horizontal_RM10mm" V 7580 6300 50  0001 C CNN
+F 2 "Resistors_ThroughHole:Resistor_Horizontal_RM15mm" V 7580 6300 50  0001 C CNN
 F 3 "" H 7650 6300 50  0000 C CNN
 	1    7650 6300
@@
 F 0 "Q1" H 8144 6050 50  0000 L CNN
 F 1 "PZT2222A" H 8144 5950 50  0000 L CNN
-F 2 "TO_SOT_Packages_SMD:SOT-223" H 8144 5850 50  0000 L CIN
+F 2 "TO_SOT_Packages_SMD:SOT-223" H 8144 5850 50  0001 L CIN
 F 3 "" H 7950 5950 50  0000 L CNN
 	1    7950 5950
 	1    0    0    -1
 $EndComp
+Wire Wire Line
+	9050 2100 9050 1950
 $EndSCHEMATC

Commit message: Updated schematics, PCB layout is nearly done.
Parts:
- D1: footprint LEDs:LED-3MM -> LEDs:LED-5MM
- R1, R10, R11, R2, R3, R4, R5, R6, R7, R8, R9: footprint Resistors_ThroughHole:Resistor_Horizontal_RM15mm -> Resistors_ThroughHole:Resistor_Horizontal_RM10mm
- Y1: footprint Crystals:Crystal_HC49-U_Horizontal_Typ1 -> Crystals:Crystal_HC49-U_Vertical
Connections:
- net GND: now also P2.5 (P5); no longer P2.6 (P6)
- net PROP_DTR: now also P2.6 (P6); no longer P2.5 (P5)
Changed lines of the file:
@@
 F 0 "R7" V 10050 5200 50  0000 C CNN
 F 1 "240" V 10000 5350 50  0000 C CNN
-F 2 "Resistors_ThroughHole:Resistor_Horizontal_RM15mm" V 9930 5350 50  0001 C CNN
+F 2 "Resistors_ThroughHole:Resistor_Horizontal_RM10mm" V 9930 5350 50  0001 C CNN
 F 3 "" H 10000 5350 50  0000 C CNN
 	1    10000 5350
@@
 F 0 "R11" V 10300 5400 50  0000 C CNN
 F 1 "240" V 10250 5250 50  0000 C CNN
-F 2 "Resistors_ThroughHole:Resistor_Horizontal_RM15mm" V 10180 5250 50  0001 C CNN
+F 2 "Resistors_ThroughHole:Resistor_Horizontal_RM10mm" V 10180 5250 50  0001 C CNN
 F 3 "" H 10250 5250 50  0000 C CNN
 	1    10250 5250
@@
 F 0 "R6" V 10050 5000 50  0000 C CNN
 F 1 "470" V 10000 5150 50  0000 C CNN
-F 2 "Resistors_ThroughHole:Resistor_Horizontal_RM15mm" V 9930 5150 50  0001 C CNN
+F 2 "Resistors_ThroughHole:Resistor_Horizontal_RM10mm" V 9930 5150 50  0001 C CNN
 F 3 "" H 10000 5150 50  0000 C CNN
 	1    10000 5150
@@
 F 0 "R10" V 10300 5200 50  0000 C CNN
 F 1 "240" V 10250 5050 50  0000 C CNN
-F 2 "Resistors_ThroughHole:Resistor_Horizontal_RM15mm" V 10180 5050 50  0001 C CNN
+F 2 "Resistors_ThroughHole:Resistor_Horizontal_RM10mm" V 10180 5050 50  0001 C CNN
 F 3 "" H 10250 5050 50  0000 C CNN
 	1    10250 5050
@@
 F 0 "R5" V 10050 4800 50  0000 C CNN
 F 1 "470" V 10000 4950 50  0000 C CNN
-F 2 "Resistors_ThroughHole:Resistor_Horizontal_RM15mm" V 9930 4950 50  0001 C CNN
+F 2 "Resistors_ThroughHole:Resistor_Horizontal_RM10mm" V 9930 4950 50  0001 C CNN
 F 3 "" H 10000 4950 50  0000 C CNN
 	1    10000 4950
@@
 F 0 "R9" V 10300 5000 50  0000 C CNN
 F 1 "240" V 10250 4850 50  0000 C CNN
-F 2 "Resistors_ThroughHole:Resistor_Horizontal_RM15mm" V 10180 4850 50  0001 C CNN
+F 2 "Resistors_ThroughHole:Resistor_Horizontal_RM10mm" V 10180 4850 50  0001 C CNN
 F 3 "" H 10250 4850 50  0000 C CNN
 	1    10250 4850
@@
 F 0 "R4" V 10050 4600 50  0000 C CNN
 F 1 "470" V 10000 4750 50  0000 C CNN
-F 2 "Resistors_ThroughHole:Resistor_Horizontal_RM15mm" V 9930 4750 50  0001 C CNN
+F 2 "Resistors_ThroughHole:Resistor_Horizontal_RM10mm" V 9930 4750 50  0001 C CNN
 F 3 "" H 10000 4750 50  0000 C CNN
 	1    10000 4750
@@
 F 0 "R8" V 10300 4800 50  0000 C CNN
 F 1 "240" V 10250 4650 50  0000 C CNN
-F 2 "Resistors_ThroughHole:Resistor_Horizontal_RM15mm" V 10180 4650 50  0001 C CNN
+F 2 "Resistors_ThroughHole:Resistor_Horizontal_RM10mm" V 10180 4650 50  0001 C CNN
 F 3 "" H 10250 4650 50  0000 C CNN
 	1    10250 4650
@@
 F 0 "Y1" H 10000 5650 50  0000 C CNN
 F 1 "5MHz" H 10000 5400 50  0000 C CNN
-F 2 "Crystals:Crystal_HC49-U_Horizontal_Typ1" H 10000 5550 50  0001 C CNN
+F 2 "Crystals:Crystal_HC49-U_Vertical" H 10000 5550 50  0001 C CNN
 F 3 "" H 10000 5550 50  0000 C CNN
 	1    10000 5550
@@
 F 0 "R3" V 9355 1950 50  0000 C CNN
 F 1 "10k" V 9455 1950 50  0000 C CNN
-F 2 "Resistors_ThroughHole:Resistor_Horizontal_RM15mm" V 9480 1950 50  0001 C CNN
+F 2 "Resistors_ThroughHole:Resistor_Horizontal_RM10mm" V 9480 1950 50  0001 C CNN
 F 3 "" H 9550 1950 50  0000 C CNN
 	1    9550 1950
@@
 F 0 "D1" V 7450 2692 50  0000 R CNN
 F 1 "LED" V 7350 2692 50  0000 R CNN
-F 2 "LEDs:LED-3MM" H 7400 2800 50  0001 C CNN
+F 2 "LEDs:LED-5MM" H 7400 2800 50  0001 C CNN
 F 3 "" H 7400 2800 50  0000 C CNN
 	1    7400 2800
@@
 F 0 "R2" V 7655 3100 50  0000 C CNN
 F 1 "1.5k" V 7755 3100 50  0000 C CNN
-F 2 "Resistors_ThroughHole:Resistor_Horizontal_RM15mm" V 7780 3100 50  0001 C CNN
+F 2 "Resistors_ThroughHole:Resistor_Horizontal_RM10mm" V 7780 3100 50  0001 C CNN
 F 3 "" H 7850 3100 50  0000 C CNN
 	1    7850 3100
@@
 F 0 "R1" V 7455 6300 50  0000 C CNN
 F 1 "10k" V 7555 6300 50  0000 C CNN
-F 2 "Resistors_ThroughHole:Resistor_Horizontal_RM15mm" V 7580 6300 50  0001 C CNN
+F 2 "Resistors_ThroughHole:Resistor_Horizontal_RM10mm" V 7580 6300 50  0001 C CNN
 F 3 "" H 7650 6300 50  0000 C CNN
 	1    7650 6300
@@
 $EndComp
 Text GLabel 10700 1850 0    60   Input ~ 0
+PROP_DTR
+Text GLabel 10350 1750 0    60   Input ~ 0
 GND
-Text GLabel 10350 1750 0    60   Input ~ 0
-PROP_DTR
 Text GLabel 10700 1650 0    60   Input ~ 0
 PROP_RX

Commit message: Production ready VGA board.
Connections:
- net PROP_RX: no longer P1.19 (P19), P2.3 (P3), U1.34 (P25), U1.39 (P30)
- net at U1.33 (P24): now also P1.17 (P17); no longer P1.20 (P20)
- net at P1.18 (P18): now also U1.34 (P25); no longer U1.35 (P26)
- net at U1.36 (P27): now also P1.20 (P20); no longer P1.17 (P17)
- new net: P1.19 (P19), U1.35 (P26)
- new net PROP_TX: P2.3 (P3), U1.39 (P30)
Other:
- moved on the sheet: C1, D1, P1, P2, P3, Q1, R1, R10, R11, R2, R3, R4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
